Commit message: complete urdf

File: tail/urdf/tail.urdf (robot description, URDF)
Before this commit: robot tail, 11 links, 10 joints
Links:
- added link link2-virtual
- added link link3-virtual
- added link link4-virtual
- added link link5-virtual
- added link link6-virtual
- added link link7-virtual
- added link link8-virtual
- added link link9-virtual
Joints:
- added joint joint2-virtual: type continuous, parent link1, child link2-virtual, origin xyz=0.0 0 0 rpy=0 0 0, axis 0 1 0
- added joint joint3-virtual: type continuous, parent link2, child link3-virtual, origin xyz=0.0 0 0 rpy=0 0 0, axis 0 1 0
- added joint joint4-virtual: type continuous, parent link3, child link4-virtual, origin xyz=0.0 0 0 rpy=0 0 0, axis 0 1 0
- added joint joint5-virtual: type continuous, parent link4, child link5-virtual, origin xyz=0.0 0 0 rpy=0 0 0, axis 0 1 0
- added joint joint6-virtual: type continuous, parent link5, child link6-virtual, origin xyz=0.0 0 0 rpy=0 0 0, axis 0 1 0
- added joint joint7-virtual: type continuous, parent link6, child link7-virtual, origin xyz=0.0 0 0 rpy=0 0 0, axis 0 1 0
- added joint joint8-virtual: type continuous, parent link7, child link8-virtual, origin xyz=0.0 0 0 rpy=0 0 0, axis 0 1 0
- added joint joint9-virtual: type continuous, parent link8, child link9-virtual, origin xyz=0.0 0 0 rpy=0 0 0, axis 0 1 0
- joint joint2: axis 1 0 0 -> 0 0 1; parent link1 -> link2-virtual
- joint joint3: axis 1 0 0 -> 0 0 1; parent link2 -> link3-virtual
- joint joint4: axis 1 0 0 -> 0 0 1; parent link3 -> link4-virtual
- joint joint5: axis 1 0 0 -> 0 0 1; parent link4 -> link5-virtual
- joint joint6: axis 1 0 0 -> 0 0 1; parent link5 -> link6-virtual
- joint joint7: axis 1 0 0 -> 0 0 1; parent link6 -> link7-virtual
- joint joint8: axis 1 0 0 -> 0 0 1; parent link7 -> link8-virtual
- joint joint9: axis 1 0 0 -> 0 0 1; parent link8 -> link9-virtual

File: tail/urdf/tail.xacro (robot description, xacro)
@@ -42,4 +42,5 @@
     </collision>
   </link>
+  <link name="link2-virtual"/>
   <link name="link2">
     <inertial>
@@ -62,4 +63,5 @@
     </collision>
   </link>
+  <link name="link3-virtual"/>
   <link name="link3">
     <inertial>
@@ -82,4 +84,5 @@
     </collision>
   </link>
+  <link name="link4-virtual"/>
   <link name="link4">
     <inertial>
@@ -102,4 +105,5 @@
     </collision>
   </link>
+  <link name="link5-virtual"/>
   <link name="link5">
     <inertial>
@@ -122,4 +126,5 @@
     </collision>
   </link>
+  <link name="link6-virtual"/>
   <link name="link6">
     <inertial>
@@ -142,4 +147,5 @@
     </collision>
   </link>
+  <link name="link7-virtual"/>
   <link name="link7">
     <inertial>
@@ -162,4 +168,5 @@
     </collision>
   </link>
+  <link name="link8-virtual"/>
   <link name="link8">
     <inertial>
@@ -182,4 +189,5 @@
     </collision>
   </link>
+  <link name="link9-virtual"/>
   <link name="link9">
     <inertial>
@@ -216,58 +224,114 @@
     <origin xyz="0.03 0.0 0.0" rpy="0.0 -0.0 0.0"/>
   </joint>
+  <joint name="joint2-virtual" type="continuous">
+    <limit effort="0.0" velocity="0.0"/>
+    <parent link="link1"/>
+    <child link="link2-virtual"/>
+    <axis xyz="0. 1. 0."/>
+    <origin xyz="0.0 0.0 0.0" rpy="0.0 -0.0 0.0"/>
+  </joint>
   <joint name="joint2" type="continuous">
     <limit effort="0.0" velocity="0.0"/>
-    <parent link="link1"/>
+    <parent link="link2-virtual"/>
     <child link="link2"/>
-    <axis xyz="1. 0. 0."/>
-    <origin xyz="0.03 0.0 0.0" rpy="0.0 -0.0 0.0"/>
+    <axis xyz="0. 0. 1."/>
+    <origin xyz="0.03 0.0 0.0" rpy="0.0 -0.0 0.0"/>
+  </joint>
+  <joint name="joint3-virtual" type="continuous">
+    <limit effort="0.0" velocity="0.0"/>
+    <parent link="link2"/>
+    <child link="link3-virtual"/>
+    <axis xyz="0. 1. 0."/>
+    <origin xyz="0.0 0.0 0.0" rpy="0.0 -0.0 0.0"/>
   </joint>
   <joint name="joint3" type="continuous">
     <limit effort="0.0" velocity="0.0"/>
-    <parent link="link2"/>
+    <parent link="link3-virtual"/>
     <child link="link3"/>
-    <axis xyz="1. 0. 0."/>
-    <origin xyz="0.03 0.0 0.0" rpy="0.0 -0.0 0.0"/>
+    <axis xyz="0. 0. 1."/>
+    <origin xyz="0.03 0.0 0.0" rpy="0.0 -0.0 0.0"/>
+  </joint>
+  <joint name="joint4-virtual" type="continuous">
+    <limit effort="0.0" velocity="0.0"/>
+    <parent link="link3"/>
+    <child link="link4-virtual"/>
+    <axis xyz="0. 1. 0."/>
+    <origin xyz="0.0 0.0 0.0" rpy="0.0 -0.0 0.0"/>
   </joint>
   <joint name="joint4" type="continuous">
     <limit effort="0.0" velocity="0.0"/>
-    <parent link="link3"/>
+    <parent link="link4-virtual"/>
     <child link="link4"/>
-    <axis xyz="1. 0. 0."/>
-    <origin xyz="0.03 0.0 0.0" rpy="0.0 -0.0 0.0"/>
+    <axis xyz="0. 0. 1."/>
+    <origin xyz="0.03 0.0 0.0" rpy="0.0 -0.0 0.0"/>
+  </joint>
+  <joint name="joint5-virtual" type="continuous">
+    <limit effort="0.0" velocity="0.0"/>
+    <parent link="link4"/>
+    <child link="link5-virtual"/>
+    <axis xyz="0. 1. 0."/>
+    <origin xyz="0.0 0.0 0.0" rpy="0.0 -0.0 0.0"/>
   </joint>
   <joint name="joint5" type="continuous">
     <limit effort="0.0" velocity="0.0"/>
-    <parent link="link4"/>
+    <parent link="link5-virtual"/>
     <child link="link5"/>
-    <axis xyz="1. 0. 0."/>
-    <origin xyz="0.03 0.0 0.0" rpy="0.0 -0.0 0.0"/>
+    <axis xyz="0. 0. 1."/>
+    <origin xyz="0.03 0.0 0.0" rpy="0.0 -0.0 0.0"/>
+  </joint>
+  <joint name="joint6-virtual" type="continuous">
+    <limit effort="0.0" velocity="0.0"/>
+    <parent link="link5"/>
+    <child link="link6-virtual"/>
+    <axis xyz="0. 1. 0."/>
+    <origin xyz="0.0 0.0 0.0" rpy="0.0 -0.0 0.0"/>
   </joint>
   <joint name="joint6" type="continuous">
     <limit effort="0.0" velocity="0.0"/>
-    <parent link="link5"/>
+    <parent link="link6-virtual"/>
     <child link="link6"/>
-    <axis xyz="1. 0. 0."/>
-    <origin xyz="0.03 0.0 0.0" rpy="0.0 -0.0 0.0"/>
+    <axis xyz="0. 0. 1."/>
+    <origin xyz="0.03 0.0 0.0" rpy="0.0 -0.0 0.0"/>
+  </joint>
+  <joint name="joint7-virtual" type="continuous">
+    <limit effort="0.0" velocity="0.0"/>
+    <parent link="link6"/>
+    <child link="link7-virtual"/>
+    <axis xyz="0. 1. 0."/>
+    <origin xyz="0.0 0.0 0.0" rpy="0.0 -0.0 0.0"/>
   </joint>
   <joint name="joint7" type="continuous">
     <limit effort="0.0" velocity="0.0"/>
-    <parent link="link6"/>
+    <parent link="link7-virtual"/>
     <child link="link7"/>
-    <axis xyz="1. 0. 0."/>
-    <origin xyz="0.03 0.0 0.0" rpy="0.0 -0.0 0.0"/>
+    <axis xyz="0. 0. 1."/>
+    <origin xyz="0.03 0.0 0.0" rpy="0.0 -0.0 0.0"/>
+  </joint>
+  <joint name="joint8-virtual" type="continuous">
+    <limit effort="0.0" velocity="0.0"/>
+    <parent link="link7"/>
+    <child link="link8-virtual"/>
+    <axis xyz="0. 1. 0."/>
+    <origin xyz="0.0 0.0 0.0" rpy="0.0 -0.0 0.0"/>
   </joint>
   <joint name="joint8" type="continuous">
     <limit effort="0.0" velocity="0.0"/>
-    <parent link="link7"/>
+    <parent link="link8-virtual"/>
     <child link="link8"/>
-    <axis xyz="1. 0. 0."/>
-    <origin xyz="0.03 0.0 0.0" rpy="0.0 -0.0 0.0"/>
+    <axis xyz="0. 0. 1."/>
+    <origin xyz="0.03 0.0 0.0" rpy="0.0 -0.0 0.0"/>
+  </joint>
+  <joint name="joint9-virtual" type="continuous">
+    <limit effort="0.0" velocity="0.0"/>
+    <parent link="link8"/>
+    <child link="link9-virtual"/>
+    <axis xyz="0. 1. 0."/>
+    <origin xyz="0.0 0.0 0.0" rpy="0.0 -0.0 0.0"/>
   </joint>
   <joint name="joint9" type="continuous">
     <limit effort="0.0" velocity="0.0"/>
-    <parent link="link8"/>
+    <parent link="link9-virtual"/>
     <child link="link9"/>
-    <axis xyz="1. 0. 0."/>
+    <axis xyz="0. 0. 1."/>
     <origin xyz="0.03 0.0 0.0" rpy="0.0 -0.0 0.0"/>
   </joint>

Commit message: add limit

File: tail/urdf/tail.urdf (robot description, URDF)
Before this commit: robot tail, 19 links, 18 joints
Joints:
- joint joint1: limit (none) -> lower=-0.78539816339 upper=0.78539816339 effort=30 velocity=0.78539816339; type continuous -> revolute
- joint joint1-virtual: limit (none) -> lower=-0.78539816339 upper=0.78539816339 effort=30 velocity=0.78539816339; type continuous -> revolute
- joint joint2: limit (none) -> lower=-0.78539816339 upper=0.78539816339 effort=30 velocity=0.78539816339; type continuous -> revolute
- joint joint2-virtual: limit (none) -> lower=-0.78539816339 upper=0.78539816339 effort=30 velocity=0.78539816339; type continuous -> revolute
- joint joint3: limit (none) -> lower=-0.78539816339 upper=0.78539816339 effort=30 velocity=0.78539816339; type continuous -> revolute
- joint joint3-virtual: limit (none) -> lower=-0.78539816339 upper=0.78539816339 effort=30 velocity=0.78539816339; type continuous -> revolute
- joint joint4: limit (none) -> lower=-0.78539816339 upper=0.78539816339 effort=30 velocity=0.78539816339; type continuous -> revolute
- joint joint4-virtual: limit (none) -> lower=-0.78539816339 upper=0.78539816339 effort=30 velocity=0.78539816339; type continuous -> revolute
- joint joint5: limit (none) -> lower=-0.78539816339 upper=0.78539816339 effort=30 velocity=0.78539816339; type continuous -> revolute
- joint joint5-virtual: limit (none) -> lower=-0.78539816339 upper=0.78539816339 effort=30 velocity=0.78539816339; type continuous -> revolute
- joint joint6: limit (none) -> lower=-0.78539816339 upper=0.78539816339 effort=30 velocity=0.78539816339; type continuous -> revolute
- joint joint6-virtual: limit (none) -> lower=-0.78539816339 upper=0.78539816339 effort=30 velocity=0.78539816339; type continuous -> revolute
- joint joint7: limit (none) -> lower=-0.78539816339 upper=0.78539816339 effort=30 velocity=0.78539816339; type continuous -> revolute
- joint joint7-virtual: limit (none) -> lower=-0.78539816339 upper=0.78539816339 effort=30 velocity=0.78539816339; type continuous -> revolute
- joint joint8: limit (none) -> lower=-0.78539816339 upper=0.78539816339 effort=30 velocity=0.78539816339; type continuous -> revolute
- joint joint8-virtual: limit (none) -> lower=-0.78539816339 upper=0.78539816339 effort=30 velocity=0.78539816339; type continuous -> revolute
- joint joint9: limit (none) -> lower=-0.78539816339 upper=0.78539816339 effort=30 velocity=0.78539816339; type continuous -> revolute
- joint joint9-virtual: limit (none) -> lower=-0.78539816339 upper=0.78539816339 effort=30 velocity=0.78539816339; type continuous -> revolute

File: tail/urdf/tail.xacro (robot description, xacro)
@@ -210,6 +210,6 @@
     </collision>
   </link>
-  <joint name="joint1-virtual" type="continuous">
-    <limit effort="0.0" velocity="0.0"/>
+  <joint name="joint1-virtual" type="revolute">
+    <limit effort="30.0" velocity="0.78539816339" lower="-0.78539816339" upper="0.78539816339"/>
     <parent link="base_link"/>
     <child link="link1-virtual"/>
@@ -217,6 +217,6 @@
     <origin xyz="0.0 0.0 0.0" rpy="0.0 -0.0 0.0"/>
   </joint>
-  <joint name="joint1" type="continuous">
-    <limit effort="0.0" velocity="0.0"/>
+  <joint name="joint1" type="revolute">
+    <limit effort="30.0" velocity="0.78539816339" lower="-0.78539816339" upper="0.78539816339"/>
     <parent link="link1-virtual"/>
     <child link="link1"/>
@@ -224,6 +224,6 @@
     <origin xyz="0.03 0.0 0.0" rpy="0.0 -0.0 0.0"/>
   </joint>
-  <joint name="joint2-virtual" type="continuous">
-    <limit effort="0.0" velocity="0.0"/>
+  <joint name="joint2-virtual" type="revolute">
+    <limit effort="30.0" velocity="0.78539816339" lower="-0.78539816339" upper="0.78539816339"/>
     <parent link="link1"/>
     <child link="link2-virtual"/>
@@ -231,6 +231,6 @@
     <origin xyz="0.0 0.0 0.0" rpy="0.0 -0.0 0.0"/>
   </joint>
-  <joint name="joint2" type="continuous">
-    <limit effort="0.0" velocity="0.0"/>
+  <joint name="joint2" type="revolute">
+    <limit effort="30.0" velocity="0.78539816339" lower="-0.78539816339" upper="0.78539816339"/>
     <parent link="link2-virtual"/>
     <child link="link2"/>
@@ -238,6 +238,6 @@
     <origin xyz="0.03 0.0 0.0" rpy="0.0 -0.0 0.0"/>
   </joint>
-  <joint name="joint3-virtual" type="continuous">
-    <limit effort="0.0" velocity="0.0"/>
+  <joint name="joint3-virtual" type="revolute">
+    <limit effort="30.0" velocity="0.78539816339" lower="-0.78539816339" upper="0.78539816339"/>
     <parent link="link2"/>
     <child link="link3-virtual"/>
@@ -245,6 +245,6 @@
     <origin xyz="0.0 0.0 0.0" rpy="0.0 -0.0 0.0"/>
   </joint>
-  <joint name="joint3" type="continuous">
-    <limit effort="0.0" velocity="0.0"/>
+  <joint name="joint3" type="revolute">
+    <limit effort="30.0" velocity="0.78539816339" lower="-0.78539816339" upper="0.78539816339"/>
     <parent link="link3-virtual"/>
     <child link="link3"/>
@@ -252,6 +252,6 @@
     <origin xyz="0.03 0.0 0.0" rpy="0.0 -0.0 0.0"/>
   </joint>
-  <joint name="joint4-virtual" type="continuous">
-    <limit effort="0.0" velocity="0.0"/>
+  <joint name="joint4-virtual" type="revolute">
+    <limit effort="30.0" velocity="0.78539816339" lower="-0.78539816339" upper="0.78539816339"/>
     <parent link="link3"/>
     <child link="link4-virtual"/>
@@ -259,6 +259,6 @@
     <origin xyz="0.0 0.0 0.0" rpy="0.0 -0.0 0.0"/>
   </joint>
-  <joint name="joint4" type="continuous">
-    <limit effort="0.0" velocity="0.0"/>
+  <joint name="joint4" type="revolute">
+    <limit effort="30.0" velocity="0.78539816339" lower="-0.78539816339" upper="0.78539816339"/>
     <parent link="link4-virtual"/>
     <child link="link4"/>
@@ -266,6 +266,6 @@
     <origin xyz="0.03 0.0 0.0" rpy="0.0 -0.0 0.0"/>
   </joint>
-  <joint name="joint5-virtual" type="continuous">
-    <limit effort="0.0" velocity="0.0"/>
+  <joint name="joint5-virtual" type="revolute">
+    <limit effort="30.0" velocity="0.78539816339" lower="-0.78539816339" upper="0.78539816339"/>
     <parent link="link4"/>
     <child link="link5-virtual"/>
@@ -273,6 +273,6 @@
     <origin xyz="0.0 0.0 0.0" rpy="0.0 -0.0 0.0"/>
   </joint>
-  <joint name="joint5" type="continuous">
-    <limit effort="0.0" velocity="0.0"/>
+  <joint name="joint5" type="revolute">
+    <limit effort="30.0" velocity="0.78539816339" lower="-0.78539816339" upper="0.78539816339"/>
     <parent link="link5-virtual"/>
     <child link="link5"/>
@@ -280,6 +280,6 @@
     <origin xyz="0.03 0.0 0.0" rpy="0.0 -0.0 0.0"/>
   </joint>
-  <joint name="joint6-virtual" type="continuous">
-    <limit effort="0.0" velocity="0.0"/>
+  <joint name="joint6-virtual" type="revolute">
+    <limit effort="30.0" velocity="0.78539816339" lower="-0.78539816339" upper="0.78539816339"/>
     <parent link="link5"/>
     <child link="link6-virtual"/>
@@ -287,6 +287,6 @@
     <origin xyz="0.0 0.0 0.0" rpy="0.0 -0.0 0.0"/>
   </joint>
-  <joint name="joint6" type="continuous">
-    <limit effort="0.0" velocity="0.0"/>
+  <joint name="joint6" type="revolute">
+    <limit effort="30.0" velocity="0.78539816339" lower="-0.78539816339" upper="0.78539816339"/>
     <parent link="link6-virtual"/>
     <child link="link6"/>
@@ -294,6 +294,6 @@
     <origin xyz="0.03 0.0 0.0" rpy="0.0 -0.0 0.0"/>
   </joint>
-  <joint name="joint7-virtual" type="continuous">
-    <limit effort="0.0" velocity="0.0"/>
+  <joint name="joint7-virtual" type="revolute">
+    <limit effort="30.0" velocity="0.78539816339" lower="-0.78539816339" upper="0.78539816339"/>
     <parent link="link6"/>
     <child link="link7-virtual"/>
@@ -301,6 +301,6 @@
     <origin xyz="0.0 0.0 0.0" rpy="0.0 -0.0 0.0"/>
   </joint>
-  <joint name="joint7" type="continuous">
-    <limit effort="0.0" velocity="0.0"/>
+  <joint name="joint7" type="revolute">
+    <limit effort="30.0" velocity="0.78539816339" lower="-0.78539816339" upper="0.78539816339"/>
     <parent link="link7-virtual"/>
     <child link="link7"/>
@@ -308,6 +308,6 @@
     <origin xyz="0.03 0.0 0.0" rpy="0.0 -0.0 0.0"/>
   </joint>
-  <joint name="joint8-virtual" type="continuous">
-    <limit effort="0.0" velocity="0.0"/>
+  <joint name="joint8-virtual" type="revolute">
+    <limit effort="30.0" velocity="0.78539816339" lower="-0.78539816339" upper="0.78539816339"/>
     <parent link="link7"/>
     <child link="link8-virtual"/>
@@ -315,6 +315,6 @@
     <origin xyz="0.0 0.0 0.0" rpy="0.0 -0.0 0.0"/>
   </joint>
-  <joint name="joint8" type="continuous">
-    <limit effort="0.0" velocity="0.0"/>
+  <joint name="joint8" type="revolute">
+    <limit effort="30.0" velocity="0.78539816339" lower="-0.78539816339" upper="0.78539816339"/>
     <parent link="link8-virtual"/>
     <child link="link8"/>
@@ -322,6 +322,6 @@
     <origin xyz="0.03 0.0 0.0" rpy="0.0 -0.0 0.0"/>
   </joint>
-  <joint name="joint9-virtual" type="continuous">
-    <limit effort="0.0" velocity="0.0"/>
+  <joint name="joint9-virtual" type="revolute">
+    <limit effort="30.0" velocity="0.78539816339" lower="-0.78539816339" upper="0.78539816339"/>
     <parent link="link8"/>
     <child link="link9-virtual"/>
@@ -329,6 +329,6 @@
     <origin xyz="0.0 0.0 0.0" rpy="0.0 -0.0 0.0"/>
   </joint>
-  <joint name="joint9" type="continuous">
-    <limit effort="0.0" velocity="0.0"/>
+  <joint name="joint9" type="revolute">
+    <limit effort="30.0" velocity="0.78539816339" lower="-0.78539816339" upper="0.78539816339"/>
     <parent link="link9-virtual"/>
     <child link="link9"/>

Commit message: wip

File: tail/urdf/tail.urdf (robot description, URDF)
Before this commit: robot tail, 19 links, 18 joints
Joints:
- joint joint1: limit lower=-0.78539816339 upper=0.78539816339 effort=30 velocity=0.78539816339 -> lower=-0.78539816339 upper=0.78539816339 effort=0.48 velocity=2
- joint joint1-virtual: limit lower=-0.78539816339 upper=0.78539816339 effort=30 velocity=0.78539816339 -> lower=-0.78539816339 upper=0.78539816339 effort=0.48 velocity=2
- joint joint2: limit lower=-0.78539816339 upper=0.78539816339 effort=30 velocity=0.78539816339 -> lower=-0.78539816339 upper=0.78539816339 effort=0.48 velocity=2
- joint joint2-virtual: limit lower=-0.78539816339 upper=0.78539816339 effort=30 velocity=0.78539816339 -> lower=-0.78539816339 upper=0.78539816339 effort=0.48 velocity=2
- joint joint3: limit lower=-0.78539816339 upper=0.78539816339 effort=30 velocity=0.78539816339 -> lower=-0.78539816339 upper=0.78539816339 effort=0.48 velocity=2
- joint joint3-virtual: limit lower=-0.78539816339 upper=0.78539816339 effort=30 velocity=0.78539816339 -> lower=-0.78539816339 upper=0.78539816339 effort=0.48 velocity=2
- joint joint4: limit lower=-0.78539816339 upper=0.78539816339 effort=30 velocity=0.78539816339 -> lower=-0.78539816339 upper=0.78539816339 effort=0.48 velocity=2
- joint joint4-virtual: limit lower=-0.78539816339 upper=0.78539816339 effort=30 velocity=0.78539816339 -> lower=-0.78539816339 upper=0.78539816339 effort=0.48 velocity=2
- joint joint5: limit lower=-0.78539816339 upper=0.78539816339 effort=30 velocity=0.78539816339 -> lower=-0.78539816339 upper=0.78539816339 effort=0.48 velocity=2
- joint joint5-virtual: limit lower=-0.78539816339 upper=0.78539816339 effort=30 velocity=0.78539816339 -> lower=-0.78539816339 upper=0.78539816339 effort=0.48 velocity=2
- joint joint6: limit lower=-0.78539816339 upper=0.78539816339 effort=30 velocity=0.78539816339 -> lower=-0.78539816339 upper=0.78539816339 effort=0.48 velocity=2
- joint joint6-virtual: limit lower=-0.78539816339 upper=0.78539816339 effort=30 velocity=0.78539816339 -> lower=-0.78539816339 upper=0.78539816339 effort=0.48 velocity=2
- joint joint7: limit lower=-0.78539816339 upper=0.78539816339 effort=30 velocity=0.78539816339 -> lower=-0.78539816339 upper=0.78539816339 effort=0.48 velocity=2
- joint joint7-virtual: limit lower=-0.78539816339 upper=0.78539816339 effort=30 velocity=0.78539816339 -> lower=-0.78539816339 upper=0.78539816339 effort=0.48 velocity=2
- joint joint8: limit lower=-0.78539816339 upper=0.78539816339 effort=30 velocity=0.78539816339 -> lower=-0.78539816339 upper=0.78539816339 effort=0.48 velocity=2
- joint joint8-virtual: limit lower=-0.78539816339 upper=0.78539816339 effort=30 velocity=0.78539816339 -> lower=-0.78539816339 upper=0.78539816339 effort=0.48 velocity=2
- joint joint9: limit lower=-0.78539816339 upper=0.78539816339 effort=30 velocity=0.78539816339 -> lower=-0.78539816339 upper=0.78539816339 effort=0.48 velocity=2
- joint joint9-virtual: limit lower=-0.78539816339 upper=0.78539816339 effort=30 velocity=0.78539816339 -> lower=-0.78539816339 upper=0.78539816339 effort=0.48 velocity=2

Commit message: send *robot* :tail :move-end-pos #f(0 0 10) worked

File: tail/urdf/tail.urdf (robot description, URDF)
Before this commit: robot tail, 19 links, 18 joints
Joints:
- joint joint1: origin xyz=0.03 0 0 rpy=0 0 0 -> xyz=0.03 0.0 0.0 rpy=0 0 0
- joint joint1-virtual: origin xyz=0.0 0 0 rpy=0 0 0 -> xyz=0 0 0 rpy=0 0 0
- joint joint2: origin xyz=0.03 0 0 rpy=0 0 0 -> xyz=0.03 0.0 0.0 rpy=0 0 0
- joint joint2-virtual: origin xyz=0.0 0 0 rpy=0 0 0 -> xyz=0 0 0 rpy=0 0 0
- joint joint3: origin xyz=0.03 0 0 rpy=0 0 0 -> xyz=0.03 0.0 0.0 rpy=0 0 0
- joint joint3-virtual: origin xyz=0.0 0 0 rpy=0 0 0 -> xyz=0 0 0 rpy=0 0 0
- joint joint4: origin xyz=0.03 0 0 rpy=0 0 0 -> xyz=0.03 0.0 0.0 rpy=0 0 0
- joint joint4-virtual: origin xyz=0.0 0 0 rpy=0 0 0 -> xyz=0 0 0 rpy=0 0 0
- joint joint5: origin xyz=0.03 0 0 rpy=0 0 0 -> xyz=0.03 0.0 0.0 rpy=0 0 0
- joint joint5-virtual: origin xyz=0.0 0 0 rpy=0 0 0 -> xyz=0 0 0 rpy=0 0 0
- joint joint6: origin xyz=0.03 0 0 rpy=0 0 0 -> xyz=0.03 0.0 0.0 rpy=0 0 0
- joint joint6-virtual: origin xyz=0.0 0 0 rpy=0 0 0 -> xyz=0 0 0 rpy=0 0 0
- joint joint7: origin xyz=0.03 0 0 rpy=0 0 0 -> xyz=0.03 0.0 0.0 rpy=0 0 0
- joint joint7-virtual: origin xyz=0.0 0 0 rpy=0 0 0 -> xyz=0 0 0 rpy=0 0 0
- joint joint8: origin xyz=0.03 0 0 rpy=0 0 0 -> xyz=0.03 0.0 0.0 rpy=0 0 0
- joint joint8-virtual: origin xyz=0.0 0 0 rpy=0 0 0 -> xyz=0 0 0 rpy=0 0 0
- joint joint9: origin xyz=0.03 0 0 rpy=0 0 0 -> xyz=0.03 0.0 0.0 rpy=0 0 0
- joint joint9-virtual: origin xyz=0.0 0 0 rpy=0 0 0 -> xyz=0 0 0 rpy=0 0 0
